Commit message: XACRO update - Added joints/links for caster wheel

File: ros2_ws/src/robot_description/urdf/patrol_robot.xacro (robot description, xacro)
@@ -1,5 +1,15 @@
 <?xml version="1.0"?>
-<robot xmlns:xacro="http://ros.org/wiki/xacro" name="patrol_bot">
-  <!-- Base Link -->
+<robot name="patrol_bot" xmlns:xacro="http://www.ros.org/wiki/xacro">
+  <!-- Materials -->
+  <material name="Gray">
+    <color rgba="0.7 0.7 0.7 1.0"/>
+  </material>
+  <material name="Black">
+    <color rgba="0.0 0.0 0.0 1.0"/>
+  </material>
+  <material name="Blue">
+    <color rgba="0.0 0.0 1.0 1.0"/>
+  </material>
+  <!-- base link -->
   <link name="base_link">
     <visual>
@@ -7,5 +17,5 @@
         <cylinder radius="0.15" length="0.05"/>
       </geometry>
-      <material name="gray"/>
+      <material name="Gray"/>
     </visual>
     <collision>
@@ -15,12 +25,11 @@
     </collision>
     <inertial>
-      <mass value="5.0"/>
-      <origin xyz="0 0 0" rpy="0 0 0"/>
-      <inertia ixx="0.1" ixy="0.0" ixz="0.0"
-               iyy="0.1" iyz="0.0"
-               izz="0.1"/>
+      <mass value="2.0"/>
+      <inertia ixx="0.01" ixy="0.0" ixz="0.0"
+               iyy="0.01" iyz="0.0"
+               izz="0.02"/>
     </inertial>
   </link>
-  <!-- Left Wheel -->
+  <!--left wheel -->
   <link name="left_wheel_link">
     <visual>
@@ -29,5 +38,5 @@
       </geometry>
       <origin xyz="0 0 0" rpy="1.5708 0 0"/>
-      <material name="black"/>
+      <material name="Black"/>
     </visual>
     <collision>
@@ -39,5 +48,4 @@
     <inertial>
       <mass value="0.2"/>
-      <origin xyz="0 0 0" rpy="0 0 0"/>
       <inertia ixx="0.001" ixy="0.0" ixz="0.0"
                iyy="0.001" iyz="0.0"
@@ -45,5 +53,5 @@
     </inertial>
   </link>
-  <!-- Right Wheel -->
+  <!-- right wheel -->
   <link name="right_wheel_link">
     <visual>
@@ -52,5 +60,5 @@
       </geometry>
       <origin xyz="0 0 0" rpy="1.5708 0 0"/>
-      <material name="black"/>
+      <material name="Black"/>
     </visual>
     <collision>
@@ -62,5 +70,4 @@
     <inertial>
       <mass value="0.2"/>
-      <origin xyz="0 0 0" rpy="0 0 0"/>
       <inertia ixx="0.001" ixy="0.0" ixz="0.0"
                iyy="0.001" iyz="0.0"
@@ -68,19 +75,25 @@
     </inertial>
   </link>
-  <!-- Left Wheel Joint -->
-  <joint name="left_wheel_joint" type="continuous">
-    <parent link="base_link"/>
-    <child link="left_wheel_link"/>
-    <origin xyz="0.0 0.1 0.025" rpy="0 0 0"/>
-    <axis xyz="0 1 0"/>
-  </joint>
-  <!-- Right Wheel Joint -->
-  <joint name="right_wheel_joint" type="continuous">
-    <parent link="base_link"/>
-    <child link="right_wheel_link"/>
-    <origin xyz="0.0 -0.1 0.025" rpy="0 0 0"/>
-    <axis xyz="0 1 0"/>
-  </joint>
-  <!-- LIDAR link -->
+  <!-- caster wheel -->
+  <link name="caster_wheel_link">
+    <visual>
+      <geometry>
+        <sphere radius="0.025"/> <!-- smaller than before -->
+      </geometry>
+      <material name="Black"/>
+    </visual>
+    <collision>
+      <geometry>
+        <sphere radius="0.025"/>
+      </geometry>
+    </collision>
+    <inertial>
+      <mass value="0.05"/>
+      <inertia ixx="0.0001" ixy="0.0" ixz="0.0"
+               iyy="0.0001" iyz="0.0"
+               izz="0.0001"/>
+    </inertial>
+  </link>
+  <!-- Gazebo lidar sensor  -->
   <link name="laser_link">
     <visual>
@@ -88,6 +101,5 @@
         <cylinder radius="0.03" length="0.05"/>
       </geometry>
-      <origin xyz="0 0 0" rpy="0 0 0"/>
-      <material name="blue"/>
+      <material name="Blue"/>
     </visual>
     <collision>
@@ -95,9 +107,7 @@
         <cylinder radius="0.03" length="0.05"/>
       </geometry>
-      <origin xyz="0 0 0" rpy="0 0 0"/>
     </collision>
     <inertial>
       <mass value="0.1"/>
-      <origin xyz="0 0 0" rpy="0 0 0"/>
       <inertia ixx="0.0001" ixy="0.0" ixz="0.0"
                iyy="0.0001" iyz="0.0"
@@ -105,32 +115,26 @@
     </inertial>
   </link>
+  <!-- Joints -->
+  <joint name="left_wheel_joint" type="continuous">
+    <parent link="base_link"/>
+    <child link="left_wheel_link"/>
+    <origin xyz="0 0.15 0" rpy="0 0 0"/>
+    <axis xyz="0 1 0"/>
+  </joint>
+  <joint name="right_wheel_joint" type="continuous">
+    <parent link="base_link"/>
+    <child link="right_wheel_link"/>
+    <origin xyz="0 -0.15 0" rpy="0 0 0"/>
+    <axis xyz="0 1 0"/>
+  </joint>
+  <joint name="caster_wheel_joint" type="fixed">
+    <parent link="base_link"/>
+    <child link="caster_wheel_link"/>
+    <origin xyz="-0.1 0 -0.025" rpy="0 0 0"/>
+  </joint>
   <joint name="laser_joint" type="fixed">
     <parent link="base_link"/>
     <child link="laser_link"/>
-    <origin xyz="0 0 0.2" rpy="0 0 0"/>
+    <origin xyz="0 0 0.08" rpy="0 0 0"/>
   </joint>
-  <!-- Gazebo lidar plugin -->
-  <gazebo>
-    <sensor type="ray" name="laser">
-      <pose>0 0 0 0 0 0</pose>
-      <ray>
-        <scan>
-          <horizontal>
-            <samples>360</samples>
-            <resolution>1</resolution>
-            <min_angle>-1.5708</min_angle>
-            <max_angle>1.5708</max_angle>
-          </horizontal>
-        </scan>
-        <range>
-          <min>0.12</min>
-          <max>10.0</max>
-        </range>
-      </ray>
-      <plugin filename="libgazebo_ros_laser.so" name="gazebo_ros_laser">
-        <topicName>/scan</topicName>
-        <frameName>laser_link</frameName>
-      </plugin>
-    </sensor>
-  </gazebo>
 </robot>
